Commit message: 1a version detección de aparcamiento

File: src/Ackermann-Autonomous-Car-Simulation/niagara_model/urdf/Autoreifen.xacro (robot description, xacro)
@@ -22,6 +22,6 @@
   <xacro:property name="degrees_90" value="1.57079633"/>
   <xacro:property name="degrees_180" value="3.14159265"/>
-  <xacro:property name="servo_stall_torque" value="75"/>  <!-- check -->
-  <xacro:property name="servo_no_load_speed" value="20"/> <!-- check -->
+  <xacro:property name="servo_stall_torque" value="100000"/>  <!-- check -->
+  <xacro:property name="servo_no_load_speed" value="1000"/> <!-- check -->
   <material name="black">
       <color rgba="0 0 0 1"/>

Commit message: Generacion path

File: src/Ackermann-Autonomous-Car-Simulation/niagara_model/urdf/Autoreifen.xacro (robot description, xacro)
@@ -62,5 +62,5 @@
       <limit lower="${-degrees_45}" upper="${degrees_45}"
             effort="${servo_stall_torque}" velocity="${servo_no_load_speed}"/>
-      <dynamics damping="10.0" friction="1.0"/>
+      <dynamics damping="0.0" friction="0.0"/>
     </joint>
     <link name="${lr_prefix}_${fr_prefix}_wheel">
