Commit message: Nuevo modelo y demas cambios

File: src/Ackermann-Autonomous-Car-Simulation/niagara_model/urdf/AckermannPlugIn.xacro (robot description, xacro)
@@ -3,12 +3,10 @@
  <!-- libgazebo_ros_ackermann_drive -->
   <gazebo>
-    <plugin name="gazebo_ros_ackermann_drive" filename="libgazebo_ros_ackermann_drive.so">
+     <plugin name="gazebo_ros_ackermann_drive" filename="libgazebo_ros_ackermann_drive.so">
       <ros>
-        <!-- <namespace></namespace> -->
         <remapping>cmd_vel:=cmd_vel</remapping>
         <remapping>odom:=odom</remapping>
       </ros>
-      <update_rate>100.0</update_rate>
-      <!-- wheels -->
+      <update_rate>500.0</update_rate>
       <front_left_joint>left_front_axle</front_left_joint>
       <front_right_joint>right_front_axle</front_right_joint>
@@ -17,19 +15,13 @@
       <left_steering_joint>left_steering_joint</left_steering_joint>
       <right_steering_joint>right_steering_joint</right_steering_joint>
-      <!-- Max absolute steer angle for tyre in radians-->
-      <!-- Any cmd_vel angular z greater than this would be capped -->
       <max_steer>1.01</max_steer>
-      <!-- Max absolute steering angle of steering wheel -->
       <max_steering_angle>6.85</max_steering_angle>
-      <!-- Max absolute linear speed in m/s -->
       <max_speed>20</max_speed>
-      <!-- PID tuning -->
-    <left_steering_pid_gain>1500 0 1</left_steering_pid_gain>
+    <left_steering_pid_gain>100000 100 10</left_steering_pid_gain>
     <left_steering_i_range>0 0</left_steering_i_range>
-    <right_steering_pid_gain>1500 0 1</right_steering_pid_gain>
+    <right_steering_pid_gain>100000 100 10</right_steering_pid_gain>
     <right_steering_i_range>0 0</right_steering_i_range>
     <linear_velocity_pid_gain>1000 0 1</linear_velocity_pid_gain>
     <linear_velocity_i_range>0 0</linear_velocity_i_range>
-      <!-- output -->
       <publish_odom>true</publish_odom>
       <publish_odom_tf>true</publish_odom_tf>

File: src/Ackermann-Autonomous-Car-Simulation/niagara_model/urdf/Autoreifen.xacro (robot description, xacro)
@@ -5,10 +5,10 @@
   <xacro:property name="hub_dia" value="0.235"/>  <!-- Reduced from 0.235 -->
   <xacro:property name="hex_hub_depth" value="0.120"/> <!-- or +0.072 -->
-  <xacro:property name="wheel_mass" value="8.0"/>   <!-- check -->
+  <xacro:property name="wheel_mass" value="0.10"/>   <!-- check -->
   <xacro:property name="wheelbase" value="2.1"/>
   <xacro:property name="hex_hub_dist" value="0.9191"/>
   <xacro:property name="wheel_travel" value="0.209492959255614"/>
-  <xacro:property name="axle_eff_limit" value="204.95"/>
-  <xacro:property name="axle_vel_limit" value="39.02"/>
+  <xacro:property name="axle_eff_limit" value="350.00"/>
+  <xacro:property name="axle_vel_limit" value="50.00"/>
   <!-- Properties of the car -->
   <xacro:property name="front_wheel_x" value="0.787346576344423"/>
@@ -94,5 +94,8 @@
     </joint>
     <gazebo reference="${lr_prefix}_${fr_prefix}_wheel">
-      <material>Gazebo/Black</material>
+       <mu1>0.01</mu1> <mu2>0.01</mu2>
+       <kp>1000000.0</kp>
+       <kd>1.0</kd>
+       <material>Gazebo/Black</material>
     </gazebo>
   </xacro:macro>
